File: pcb/v2Low/roba_L.kicad_pcb (KiCad board)
At the start: 2 copper layers, 10.7 x 12.1 mm, 56 parts, among them J1 Conn_01x01-Connector_Generic, J2 Conn_01x01-Connector_Generic, J3 Conn_01x01-Connector_Generic, J4 Conn_01x01-Connector_Generic, J5 Conn_01x01-Connector_Generic, J6 Conn_01x01-Connector_Generic, J7 Conn_01x01-Connector_Generic, SW1 SW_PUSH, SW10 SW_PUSH, SW11 SW_PUSH, SW12 SW_PUSH, SW13 SW_PUSH, SW14 SW_PUSH, SW15 SW_PUSH, SW16 SW_PUSH, SW17 SW_PUSH, SW18 SW_PUSH, SW19 SW_PUSH, SW2 SW_PUSH, SW20 SW_PUSH, SW21 SW_PUSH, SW22 SW_PUSH, SW23 SW_PUSH, SW24 SW_SPDT, SW3 SW_PUSH, SW4 SW_PUSH, SW5 SW_PUSH, SW6 SW_PUSH, SW7 SW_PUSH, SW8 SW_PUSH, SW9 SW_PUSH

Commit message: save
Parts:
- removed J1, J2, J3, J4, J5, J6, J7: Conn_01x01-Connector_Generic, MountingHole:MountingHole_4.3mm_M4
- moved SW5 80.4 mm to (67.0, 41.5)
- moved SW6 78.8 mm to (67.0, 58.5)
- moved SW17 77.6 mm to (118.0, 41.5)
- moved SW18 75.9 mm to (118.0, 58.5)
- moved SW9 59.3 mm to (84.0, 33.0)
- moved SW10 57.8 mm to (84.0, 50.0)
- moved SW11 56.2 mm to (84.0, 67.0)
- moved SW12 54.7 mm to (84.0, 84.0)
- moved SW8 43.3 mm to (67.0, 92.5)
- moved SW7 42.6 mm to (67.0, 75.5)
- moved SW13 29.7 mm to (101.0, 37.2)
- moved SW14 28.6 mm to (101.0, 54.2)
- moved SW19 28.2 mm to (118.0, 75.5)
- moved SW15 27.5 mm to (101.0, 71.2)

Commit message: save
Parts:
- moved U1 66.2 mm to (135.9, 29.1)
- moved SW20 34.1 mm to (122.0, 102.0)
- moved SW21 30.1 mm to (135.0, 58.5)
- moved SW22 28.5 mm to (135.0, 75.5)
- moved SW16 18.0 mm to (105.0, 100.0)
- moved SW23 14.9 mm to (139.0, 104.0)

Commit message: save
Parts:
- moved D1 120.6 mm to (48.0, 45.0)
- moved D5 119.7 mm to (65.0, 36.5)
- moved D2 112.8 mm to (48.0, 62.0)
- moved D9 111.9 mm to (82.0, 28.0)
- moved D6 109.4 mm to (65.0, 53.5)
- moved D13 106.5 mm to (99.0, 32.2)
- moved D3 106.4 mm to (48.0, 79.0)
- moved D4 101.8 mm to (48.0, 96.0)
- moved D10 101.0 mm to (82.0, 45.0)
- moved D7 100.3 mm to (65.0, 70.5)
- moved D14 94.2 mm to (99.0, 49.2)
- moved D8 92.5 mm to (65.0, 87.5)
- moved D11 91.1 mm to (82.0, 62.0)
- moved D17 89.2 mm to (116.0, 36.5)
- moved D12 82.7 mm to (82.0, 79.0)
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Changed lines of the file:
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@@
 	(footprint "roBa:Diode_SMD"
 		(layer "F.Cu")
-		(at 152.833125 116.965942)
+		(at 82 45)
 		(descr "https://github.com/e3w2q/su120-keyboard (diode_SMD_rev2)")
 		(property "Reference" "D10"
@@
 	(footprint "roBa:Diode_SMD"
 		(layer "F.Cu")
-		(at 159.18625 114.575314)
+		(at 116 36.5)
 		(descr "https://github.com/e3w2q/su120-keyboard (diode_SMD_rev2)")
 		(property "Reference" "D17"
@@
 	(footprint "roBa:XIAO_nRF52840_wBAT_wNFC_1"
 		(layer "F.Cu")
-		(at 135.88 29.12)
+		(at 140 25)
 		(descr "https://gitlab.com/lpgalaxy/revxlp(xiao-ble-smd)")
 		(property "Reference" "U1"
@@
 	(footprint "roBa:Diode_SMD"
 		(layer "F.Cu")
-		(at 146.48 121.747198)
+		(at 48 96)
 		(descr "https://github.com/e3w2q/su120-keyboard (diode_SMD_rev2)")
 		(property "Reference" "D4"
@@
 	(footprint "roBa:Diode_SMD"
 		(layer "F.Cu")
-		(at 146.48 116.965942)
+		(at 48 62)
 		(descr "https://github.com/e3w2q/su120-keyboard (diode_SMD_rev2)")
 		(property "Reference" "D2"
@@
 	(footprint "roBa:Diode_SMD"
 		(layer "F.Cu")
-		(at 146.48 119.35657)
+		(at 48 79)
 		(descr "https://github.com/e3w2q/su120-keyboard (diode_SMD_rev2)")
 		(property "Reference" "D3"
@@
 	(footprint "roBa:Diode_SMD"
 		(layer "F.Cu")
-		(at 146.48 128.919082)
+		(at 65 70.5)
 		(descr "https://github.com/e3w2q/su120-keyboard (diode_SMD_rev2)")
 		(property "Reference" "D7"
@@
 	(footprint "roBa:Diode_SMD"
 		(layer "F.Cu")
-		(at 146.48 114.575314)
+		(at 48 45)
 		(descr "https://github.com/e3w2q/su120-keyboard (diode_SMD_rev2)")
 		(property "Reference" "D1"
@@
 	(footprint "roBa:Diode_SMD"
 		(layer "F.Cu")
-		(at 152.833125 126.528454)
+		(at 99 49.25)
 		(descr "https://github.com/e3w2q/su120-keyboard (diode_SMD_rev2)")
 		(property "Reference" "D14"
@@
 	(footprint "roBa:Diode_SMD"
 		(layer "F.Cu")
-		(at 159.18625 128.919082)
+		(at 137 99)
 		(descr "https://github.com/e3w2q/su120-keyboard (diode_SMD_rev2)")
 		(property "Reference" "D23"
@@
 	(footprint "roBa:Diode_SMD"
 		(layer "F.Cu")
-		(at 159.18625 124.137826)
+		(at 133 53.5)
 		(descr "https://github.com/e3w2q/su120-keyboard (diode_SMD_rev2)")
 		(property "Reference" "D21"
@@
 	(footprint "roBa:Diode_SMD"
 		(layer "F.Cu")
-		(at 152.833125 128.919082)
+		(at 99 66.25)
 		(descr "https://github.com/e3w2q/su120-keyboard (diode_SMD_rev2)")
 		(property "Reference" "D15"
@@
 	(footprint "roBa:Diode_SMD"
 		(layer "F.Cu")
-		(at 152.833125 114.575314)
+		(at 82 28)
 		(descr "https://github.com/e3w2q/su120-keyboard (diode_SMD_rev2)")
 		(property "Reference" "D9"
@@
 	(footprint "roBa:Diode_SMD"
 		(layer "F.Cu")
-		(at 159.18625 119.35657)
+		(at 116 70.5)
 		(descr "https://github.com/e3w2q/su120-keyboard (diode_SMD_rev2)")
 		(property "Reference" "D19"
@@
 	(footprint "roBa:Diode_SMD"
 		(layer "F.Cu")
-		(at 152.833125 119.35657)
+		(at 82 62)
 		(descr "https://github.com/e3w2q/su120-keyboard (diode_SMD_rev2)")
 		(property "Reference" "D11"
@@
 	(footprint "roBa:Diode_SMD"
 		(layer "F.Cu")
-		(at 159.18625 121.747198)
+		(at 120 97)
 		(descr "https://github.com/e3w2q/su120-keyboard (diode_SMD_rev2)")
 		(property "Reference" "D20"
@@
 	(footprint "roBa:Diode_SMD"
 		(layer "F.Cu")
-		(at 146.48 124.137826)
+		(at 65 36.5)
 		(descr "https://github.com/e3w2q/su120-keyboard (diode_SMD_rev2)")
 		(property "Reference" "D5"
@@
 	(footprint "roBa:Diode_SMD"
 		(layer "F.Cu")
-		(at 152.833125 121.747198)
+		(at 82 79)
 		(descr "https://github.com/e3w2q/su120-keyboard (diode_SMD_rev2)")
 		(property "Reference" "D12"
@@
 	(footprint "roBa:Diode_SMD"
 		(layer "F.Cu")
-		(at 146.48 131.30971)
+		(at 65 87.5)
 		(descr "https://github.com/e3w2q/su120-keyboard (diode_SMD_rev2)")
 		(property "Reference" "D8"
@@
 	(footprint "roBa:Diode_SMD"
 		(layer "F.Cu")
-		(at 146.48 126.528454)
+		(at 65 53.5)
 		(descr "https://github.com/e3w2q/su120-keyboard (diode_SMD_rev2)")
 		(property "Reference" "D6"
@@
 	(footprint "roBa:Diode_SMD"
 		(layer "F.Cu")
-		(at 159.18625 126.528454)
+		(at 133 70.5)
 		(descr "https://github.com/e3w2q/su120-keyboard (diode_SMD_rev2)")
 		(property "Reference" "D22"
@@
 	(footprint "roBa:Diode_SMD"
 		(layer "F.Cu")
-		(at 152.833125 131.30971)
+		(at 103 95)
 		(descr "https://github.com/e3w2q/su120-keyboard (diode_SMD_rev2)")
 		(property "Reference" "D16"
@@
 	(footprint "roBa:Diode_SMD"
 		(layer "F.Cu")
-		(at 159.18625 116.965942)
+		(at 116 53.5)
 		(descr "https://github.com/e3w2q/su120-keyboard (diode_SMD_rev2)")
 		(property "Reference" "D18"
@@
 	(footprint "roBa:Diode_SMD"
 		(layer "F.Cu")
-		(at 152.833125 124.137826)
+		(at 99 32.25)
 		(descr "https://github.com/e3w2q/su120-keyboard (diode_SMD_rev2)")
 		(property "Reference" "D13"

Commit message: save
Parts:
- B1: moved to B.Cu
- moved B1 102.0 mm to (137.0, 40.0), turned to 180 degrees
- moved SW24 54.1 mm to (150.0, 80.0), turned to -90 degrees
- moved U1 5.39 mm to (138.0, 20.0)
Other:
- board size 10.7 x 12.1 mm -> 112 x 94 mm

Commit message: start R
Parts:
- moved D16 5.83 mm to (100.0, 90.0)
- moved D20 5.83 mm to (117.0, 92.0)
- moved D23 5.83 mm to (134.0, 94.0)
- moved SW16 5.83 mm to (102.0, 95.0)
- moved SW20 5.83 mm to (119.0, 97.0)
- moved SW23 5.83 mm to (136.0, 99.0)
Routing:
- net Row3: track 0.00 -> 179.1 mm, vias 0 -> 5
- net Col0: track 0.00 -> 177.8 mm, vias 0 -> 1
- net Row2: track 0.00 -> 150.4 mm, vias 0 -> 6
- net Row1: track 0.00 -> 149.3 mm, vias 0 -> 6
- net Col1: track 0.00 -> 149.3 mm, vias 0 -> 1
- net Col2: track 0.00 -> 127.9 mm, vias 0 -> 1
- net Col3: track 0.00 -> 126.1 mm, vias 0 -> 1
- net Row0: track 0.00 -> 100.8 mm
- net Col4: track 0.00 -> 95.8 mm, vias 0 -> 1
- net Col5: track 0.00 -> 75.9 mm, vias 0 -> 1
- net GND: track 0.00 -> 73.6 mm
- net Net-(B1--): track 0.00 -> 45.1 mm
- net Bat: track 0.00 -> 11.7 mm
- net Net-(D23-A): track 0.00 -> 11.3 mm
- net Net-(D22-A): track 0.00 -> 11.3 mm
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Other:
- board size 112 x 94 mm -> 112 x 91 mm
