File: pcb/v2R-Low/roba_R.kicad_sch (KiCad schematic)
At the start: 50 parts, among them J2 Conn_01x01-Connector_Generic, J3 Conn_01x01-Connector_Generic, J4 Conn_01x01-Connector_Generic, J5 Conn_01x01-Connector_Generic, J6 Conn_01x01-Connector_Generic, J7 Conn_01x01-Connector_Generic, SW1 SW_PUSH, SW10 SW_PUSH, SW11 SW_PUSH, SW12 SW_PUSH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

Commit message: 右のpcbまでok
Parts:
- SW10, SW11, SW13, SW14, SW15, SW17, SW18, SW19, SW2, SW20, SW3, SW4, SW5, SW6, SW7, SW8, SW9: footprint roBa:SW_MX -> ChocV2_Hotswap:Choc_v2_Hotswap_1u
- SW12, SW16: footprint roBa:SW_MX_Choc -> ChocV2_Hotswap:Choc_v2_Hotswap_1u
Changed lines of the file:
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@@
 			)
 		)
-		(property "Footprint" "roBa:SW_MX"
+		(property "Footprint" "ChocV2_Hotswap:Choc_v2_Hotswap_1u"
 			(at 204.47 80.01 0)
 			(effects
@@
 			)
 		)
-		(property "Footprint" "roBa:SW_MX"
+		(property "Footprint" "ChocV2_Hotswap:Choc_v2_Hotswap_1u"
 			(at 223.52 80.01 0)
 			(effects
@@
 			)
 		)
-		(property "Footprint" "roBa:SW_MX_Choc"
+		(property "Footprint" "ChocV2_Hotswap:Choc_v2_Hotswap_1u"
 			(at 223.52 97.79 0)
 			(effects
@@
 			)
 		)
-		(property "Footprint" "roBa:SW_MX"
+		(property "Footprint" "ChocV2_Hotswap:Choc_v2_Hotswap_1u"
 			(at 223.52 60.96 0)
 			(effects
@@
 			)
 		)
-		(property "Footprint" "roBa:SW_MX"
+		(property "Footprint" "ChocV2_Hotswap:Choc_v2_Hotswap_1u"
 			(at 166.37 60.96 0)
 			(effects
@@
 			)
 		)
-		(property "Footprint" "roBa:SW_MX_Choc"
+		(property "Footprint" "ChocV2_Hotswap:Choc_v2_Hotswap_1u"
 			(at 204.47 97.79 0)
 			(effects
@@
 			)
 		)
-		(property "Footprint" "roBa:SW_MX"
+		(property "Footprint" "ChocV2_Hotswap:Choc_v2_Hotswap_1u"
 			(at 166.37 80.01 0)
 			(effects
@@
 			)
 		)
-		(property "Footprint" "roBa:SW_MX"
+		(property "Footprint" "ChocV2_Hotswap:Choc_v2_Hotswap_1u"
 			(at 223.52 41.91 0)
 			(effects
@@
 			)
 		)
-		(property "Footprint" "roBa:SW_MX"
+		(property "Footprint" "ChocV2_Hotswap:Choc_v2_Hotswap_1u"
 			(at 166.37 97.79 0)
 			(effects
@@
 			)
 		)
-		(property "Footprint" "roBa:SW_MX"
+		(property "Footprint" "ChocV2_Hotswap:Choc_v2_Hotswap_1u"
 			(at 242.57 60.96 0)
 			(effects
@@
 			)
 		)
-		(property "Footprint" "roBa:SW_MX"
+		(property "Footprint" "ChocV2_Hotswap:Choc_v2_Hotswap_1u"
 			(at 204.47 41.91 0)
 			(effects
@@
 			)
 		)
-		(property "Footprint" "roBa:SW_MX"
+		(property "Footprint" "ChocV2_Hotswap:Choc_v2_Hotswap_1u"
 			(at 242.57 80.01 0)
 			(effects
@@
 			)
 		)
-		(property "Footprint" "roBa:SW_MX"
+		(property "Footprint" "ChocV2_Hotswap:Choc_v2_Hotswap_1u"
 			(at 204.47 60.96 0)
 			(effects
@@
 			)
 		)
-		(property "Footprint" "roBa:SW_MX"
+		(property "Footprint" "ChocV2_Hotswap:Choc_v2_Hotswap_1u"
 			(at 185.42 97.79 0)
 			(effects
@@
 			)
 		)
-		(property "Footprint" "roBa:SW_MX"
+		(property "Footprint" "ChocV2_Hotswap:Choc_v2_Hotswap_1u"
 			(at 242.57 97.79 0)
 			(effects
@@
 			)
 		)
-		(property "Footprint" "roBa:SW_MX"
+		(property "Footprint" "ChocV2_Hotswap:Choc_v2_Hotswap_1u"
 			(at 185.42 41.91 0)
 			(effects
@@
 			)
 		)
-		(property "Footprint" "roBa:SW_MX"
+		(property "Footprint" "ChocV2_Hotswap:Choc_v2_Hotswap_1u"
 			(at 185.42 60.96 0)
 			(effects
@@
 			)
 		)
-		(property "Footprint" "roBa:SW_MX"
+		(property "Footprint" "ChocV2_Hotswap:Choc_v2_Hotswap_1u"
 			(at 185.42 80.01 0)
 			(effects
@@
 			)
 		)
-		(property "Footprint" "roBa:SW_MX"
+		(property "Footprint" "ChocV2_Hotswap:Choc_v2_Hotswap_1u"
 			(at 242.57 41.91 0)
 			(effects
