File: pcb/v2R-Low/roba_R.kicad_pcb (KiCad board)
At the start: 2 copper layers, 10.7 x 12.1 mm, 50 parts, among them J2 Conn_01x01-Connector_Generic, J3 Conn_01x01-Connector_Generic, J4 Conn_01x01-Connector_Generic, J5 Conn_01x01-Connector_Generic, J6 Conn_01x01-Connector_Generic, J7 Conn_01x01-Connector_Generic, SW1 SW_PUSH, SW10 SW_PUSH, SW11 SW_PUSH, SW12 SW_PUSH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

Commit message: 右のpcbまでok
Parts:
- removed J2, J3, J4, J5, J6, J7: Conn_01x01-Connector_Generic, MountingHole:MountingHole_4.3mm_M4
- moved D17 138.0 mm to (248.0, 45.0)
- moved D13 137.9 mm to (231.0, 36.5)
- moved D18 131.4 mm to (248.0, 62.0)
- moved D14 129.4 mm to (231.0, 53.5)
- moved D19 126.1 mm to (248.0, 79.0)
- moved D9 124.1 mm to (214.0, 28.0)
- moved J1 123.0 mm to (234.1, 99.1)
- moved D20 122.3 mm to (248.0, 96.0)
- moved D5 118.5 mm to (197.0, 32.2)
- moved D10 114.8 mm to (214.0, 45.0)
- moved SW9 112.8 mm to (216.0, 33.0)
- moved SW10 112.5 mm to (216.0, 50.0)
- moved SW11 112.2 mm to (216.0, 67.0)
- moved SW5 112.2 mm to (199.0, 37.2)
- moved SW6 112.0 mm to (199.0, 54.2)
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Other:
- board size 10.7 x 12.1 mm -> 112 x 91 mm

Commit message: 配線までok
Routing:
- net SDIO: track 0.00 -> 174.5 mm, vias 0 -> 2
- net MOTION: track 0.00 -> 167.7 mm, vias 0 -> 1
- net GND: track 0.00 -> 166.5 mm, vias 0 -> 1
- net Row3: track 0.00 -> 165.5 mm, vias 0 -> 5
- net Col3: track 0.00 -> 161.2 mm, vias 0 -> 1
- net Row2: track 0.00 -> 159.2 mm, vias 0 -> 6
- net Col2: track 0.00 -> 151.5 mm, vias 0 -> 1
- net SCLK: track 0.00 -> 140.7 mm, vias 0 -> 1
- net Row1: track 0.00 -> 140.6 mm, vias 0 -> 6
- net Col4: track 0.00 -> 139.4 mm, vias 0 -> 1
- net Col1: track 0.00 -> 138.3 mm, vias 0 -> 3
- net 3.3V: track 0.00 -> 131.6 mm, vias 0 -> 1
- net CS: track 0.00 -> 125.4 mm, vias 0 -> 1
- net Row0: track 0.00 -> 120.3 mm, vias 0 -> 3
- net Col0: track 0.00 -> 77.3 mm, vias 0 -> 2
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